File: MK_e-LIFE.kicad_pcb (KiCad board)
At the start: 2 copper layers, 59 x 40 mm, 6 parts, among them Q1 IRG4PF50W

Commit message: up
Parts:
- added BT1: 2462, 2462:BAT_2462, F.Cu at (89.9, 84.8)
- Q1: value IRG4PF50W -> 2SC1815; footprint Package_TO_SOT_THT:TO-247-3_Vertical -> Package_TO_SOT_THT:TO-92_Inline
- R1, R2, R3: footprint Capacitor_THT:C_Radial_D5.0mm_H5.0mm_P2.00mm -> Resistor_THT:R_Axial_DIN0204_L3.6mm_D1.6mm_P7.62mm_Horizontal
- moved Q1 5.45 mm to (154.0, 107.0)
Connections:
- D1 pad 1: +3V0 -> GND
- D2 pad 2: +3V0 -> Net-(D2-A)
- Q1 pad 1: Net-(Q1-G) -> GND
- Q1 pad 3: +3V0 -> Net-(Q1-B)
- R1 pad 2: Net-(Q1-G) -> Net-(Q1-B)
- R2 pad 1: Net-(Q1-G) -> Net-(Q1-B)
- R2 pad 2: +3V0 -> GND
- R3 pad 1: +3V0 -> Net-(D2-A)
Routing:
- net +3V0: track 100.8 -> 0.00 mm
- net GND: track 0.00 -> 80.4 mm
- net Net-(D2-A): track 0.00 -> 49.6 mm
- net Net-(D1-A): track 37.3 -> 0.00 mm
- net Net-(Q1-G): track 31.4 -> 0.00 mm
- net Net-(D2-K): track 14.2 -> 0.00 mm
- added copper zone on F.Cu, net GND
Other:
- board size 59 x 40 mm -> 123 x 69 mm
