File: MK_e-LIFE.kicad_sch (KiCad schematic)
At the start: 6 parts, among them Q1 IRG4PF50W

Commit message: up
Parts:
- removed Q1: IRG4PF50W, Package_TO_SOT_THT:TO-247-3_Vertical, symbol Transistor_IGBT:IRG4PF50W
- added BT1: 2462, 2462:BAT_2462, symbol 2462:2462
- added Q1: 2SC1815, Package_TO_SOT_THT:TO-92_Inline, symbol Transistor_BJT:2SC1815
- R1, R2, R3: footprint Capacitor_THT:C_Radial_D5.0mm_H5.0mm_P2.00mm -> Resistor_THT:R_Axial_DIN0204_L3.6mm_D1.6mm_P7.62mm_Horizontal
Connections:
- net at D1.2 (A), R3.2: now also Q1.2 (C)
- net at R1.2, R2.1: now also Q1.3 (B)
- net +3V0: no longer names the net of D2.2 (A), R3.1
- net +3V0: now also BT1.P; no longer D1.1 (K), R2.2
- new net GND: BT1.N, D1.1 (K), Q1.1 (E), R2.2
